File: scintillator_field/hardware/sipm/sipm.kicad_pcb (KiCad board)
At the start: 2 copper layers, 41 x 18 mm, 13 parts, among them J1 SMA BIAS, J2 SMA SIGNAL

Commit message: finalized SiPM PCB
Parts:
- added G***: LOGO, logos:sc, F.Cu at (184.5, 91.0)
- J1: value SMA BIAS -> SMA POWER
- moved C1 1.50 mm to (161.0, 90.5)
- moved R1 1.50 mm to (159.0, 90.5)
Routing:
- net Net-(C1-Pad1): track 4.03 -> 6.03 mm
- net Net-(J1-In): track 8.45 -> 9.07 mm
