File: scintillator_field/hardware/sipm/sipm.kicad_sch (KiCad schematic)
At the start: 10 parts, among them J1 SMA POWER, J2 SMA SIGNAL

Commit message: finalized SiPM PCB
Other:
- moved on the sheet: C1, C2, C3, C4, D1, J1, J2, R1, R2, R3
