File: scintillator_field/hardware/power/power.kicad_pcb (KiCad board)
At the start: 2 copper layers, 54 x 24 mm, 21 parts, among them J1 POWER, J2 POWER, J3 POWER, J4 POWER, U1 LT3461A

Commit message: run drc
Parts:
- moved G*** 2.93 mm to (137.5, 100.0)
Other:
- board size 54 x 24 mm -> 54 x 24.4 mm

Commit message: power
Parts:
- moved G*** 2.92 mm to (137.2, 97.1)
Changed lines of the file:
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@@
 			(plot_on_all_layers_selection 0x0000000_00000000)
 			(disableapertmacros no)
-			(usegerberextensions no)
+			(usegerberextensions yes)
 			(usegerberattributes yes)
 			(usegerberadvancedattributes yes)
-			(creategerberjobfile yes)
+			(creategerberjobfile no)
 			(dashed_line_dash_ratio 12.000000)
 			(dashed_line_gap_ratio 3.000000)
@@
 			(plotinvisibletext no)
 			(sketchpadsonfab no)
-			(subtractmaskfromsilk no)
+			(subtractmaskfromsilk yes)
 			(outputformat 1)
 			(mirror no)
-			(drillshape 1)
+			(drillshape 0)
 			(scaleselection 1)
 			(outputdirectory "")
@@
 	(footprint "power:hep_20mm"
 		(layer "B.Cu")
-		(at 137.5 100 90)
+		(at 137.2 97.1 90)
 		(property "Reference" "G***"
 			(at 0 0 90)
