File: scintillator_field/hardware/v2/acquisition/acquisition/fpga.kicad_sch (KiCad schematic)
At the start: 1 part, among them U2 ICE40UP5K-SG48ITR

Commit message: Small changes on all sheets
Connections:
- net +3V3: now reaches U2.1 (VCCIO_2)
- net +3V3: now also U2.22 (SPI_VCCIO1), U2.33 (VCCIO_0)
- net +2V5: now reaches U2.24 (VPP_2V5)
- net +1V2: now reaches U2.29 (VCCPLL)
- net +1V2: now also U2.30 (VCC), U2.5 (VCC)
- net GND: now reaches U2.49 (GND)
Other:
- moved on the sheet: U2B, U2C
